File: Placa_Iot/rf_lora.kicad_sch (KiCad schematic)
At the start: 0 parts

Commit message: RF commit
Parts:
- added C22, C23, C24: NC, Capacitor_SMD:C_0402_1005Metric, symbol Device:C
- added J3: 20279-001E-03, antennas:IPEX_MHF_I, symbol antenas:IPEX_MHF_I
- added R11, R12, R13, R9: 22 Ohm, Resistor_SMD:R_0402_1005Metric, symbol resistor:R
- added U5: T-SX1262, ic_control:MODULE_T_SX1262, symbol ic_control:T_SX1262
Connections:
- new net: R13.1, U5.13 (NC)
- new net: C23.2, C24.1, J3.1 (In)
- new net: C22.1, C23.1, U5.16 (ANT)
- new net: R12.1, U5.10 (DIO1)
- new net: R11.1, U5.14 (DIO3)
- new net: R9.1, U5.9 (BUSY)
- new net +3.3V: U5.12 (3.3V)
- new net GND: C22.2, C24.2, J3.2 (Ext), J3.3 (Ext), U5.1 (GND), U5.15 (GND), U5.8 (GND)
- new net IO3: U5.7 (MISO)
- new net IO33: R12.2
- new net IO34: R9.2
- new net IO36: U5.2 (NC)
- new net IO5: U5.5 (SCK)
- new net IO6: U5.6 (MOSI)
- new net IO7: U5.4 (NSS)
- new net IO8: U5.3 (NRESET)
- new net IO9: U5.11 (NC)
- new net LORA_RX: R11.2
- new net LORA_TX: R13.2
